File: schematics/wake_on_sleep.sch (EAGLE design)
At the start: 30 parts, among them Q1 MMBT3904, Q2 MMBT3904, Q3 MMBT3904, U1 PIC16F1823ST, U2 ADP160, U3 ADXL362

Commit message: Updated to Rev A.1 and prepared for PCB build
Parts:
- BAT1: device kevin:BATTERY20SMD -> kevin:BATTERY20MM_SMD; PARTNO S8211-46R -> BA2032SM
Connections:
- net !AWAKE.OUT: now also JP2.2; no longer JP2.3
- net AWAKE.OUT: now also JP2.3; no longer JP2.2
Changed lines of the file:
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@@
 <attribute name="PARTNO" value="254-EMB140-R0"/>
 </part>
-<part name="BAT1" library="kevin" deviceset="BATTERY" device="20SMD" value="CR2032-20MM">
-<attribute name="PARTNO" value="S8211-46R"/>
+<part name="BAT1" library="kevin" deviceset="BATTERY" device="20MM_SMD" value="CR2032-20MM">
+<attribute name="PARTNO" value="BA2032SM"/>
 </part>
 <part name="LED3" library="kevin" deviceset="LED" device="CHIPLED_0603" value="GREEN">
@@
 </segment>
 <segment>
-<pinref part="JP2" gate="G$1" pin="2"/>
-<wire x1="78.74" y1="30.48" x2="73.66" y2="30.48" width="0.1524" layer="91"/>
-<label x="73.66" y="30.48" size="1.778" layer="95" rot="R180"/>
+<wire x1="78.74" y1="27.94" x2="73.66" y2="27.94" width="0.1524" layer="91"/>
+<label x="73.66" y="27.94" size="1.778" layer="95" rot="R180"/>
+<pinref part="JP2" gate="G$1" pin="3"/>
 </segment>
 </net>
@@
 </segment>
 <segment>
-<pinref part="JP2" gate="G$1" pin="3"/>
-<wire x1="78.74" y1="27.94" x2="73.66" y2="27.94" width="0.1524" layer="91"/>
-<label x="73.66" y="27.94" size="1.778" layer="95" rot="R180"/>
-</segment>
-</net>
+<wire x1="78.74" y1="30.48" x2="73.66" y2="30.48" width="0.1524" layer="91"/>
+<label x="73.66" y="30.48" size="1.778" layer="95" rot="R180"/>
+<pinref part="JP2" gate="G$1" pin="2"/>
+</segment>
+</net>
